File: noise_measurement/noise_measurement.kicad_sch (KiCad schematic)
At the start: 15 parts, among them U1 OPA344, U2 MSP430G2210ID, U3 SPH8878LR5H-2

Commit message: Add files via upload
Parts:
- added C5, C7: 0.1uF, Capacitor_SMD:C_0402_1005Metric, symbol Device:C
- added J1: Conn_01x06_Pin, Connector_PinHeader_1.27mm:PinHeader_1x06_P1.27mm_Vertical, symbol Connector:Conn_01x06_Pin
- added TP1, TP2: TestPoint, TestPoint:TestPoint_Pad_D1.0mm, symbol Connector:TestPoint
Connections:
- net GND: now also C5.1, C7.1, J1.1 (Pin_1)
- net SBTCK: now also J1.5 (Pin_5)
- net SBWTDIO: now also J1.6 (Pin_6)
- net SCL: now also J1.4 (Pin_4)
- net SDA: now also J1.3 (Pin_3)
- net VCC: now also C5.2, C7.2, J1.2 (Pin_2)
- net at C2.1, R2.1, U1.1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: now also TP1.1
- net at C2.2, R1.1, R2.2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: now also TP2.1
Other:
- moved on the sheet: C1, R1

Commit message: Add files via upload
Parts:
- TP1: value TestPoint -> op-amp OUT
- TP2: value TestPoint -> OUT(+)
Changed lines of the file:
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@@
-		)
-	)
-	(label "SDA"
-		(at 182.88 80.01 0)
-		(effects
-			(font
-				(size 1.27 1.27)
-			)
-			(justify left bottom)
 		)
 	)
@@
 	)
 	(label "SBTCK"
-		(at 113.03 92.71 0)
-		(effects
-			(font
-				(size 1.27 1.27)
-			)
-			(justify left bottom)
-		)
-	)
-	(label "SCL"
-		(at 182.88 77.47 0)
-		(effects
-			(font
-				(size 1.27 1.27)
-			)
-			(justify left bottom)
-		)
-	)
-	(label "GND"
-		(at 113.03 100.33 0)
-		(effects
-			(font
-				(size 1.27 1.27)
-			)
-			(justify left bottom)
-		)
-	)
-	(label "3.3V"
-		(at 113.03 96.52 0)
-		(effects
-			(font
-				(size 1.27 1.27)
-			)
-			(justify left bottom)
-		)
-	)
-	(label "SBWTDIO"
-		(at 113.03 88.9 0)
-		(effects
-			(font
-				(size 1.27 1.27)
-			)
-			(justify left bottom)
-		)
-	)
-	(label "SBTCK"
 		(at 68.58 118.11 0)
 		(effects
@@
 			)
 		)
-		(property "Value" "TestPoint"
+		(property "Value" "OUT(+)"
 			(at 82.55 38.6079 0)
 			(show_name no)
@@
 			)
 		)
-		(property "Value" "TestPoint"
+		(property "Value" "op-amp OUT"
 			(at 132.08 42.4179 0)
 			(show_name no)

Commit message: Add files via upload
Connections:
- net SBWTDIO: now also J1.5 (Pin_5); no longer J1.6 (Pin_6)
- net SBTCK renamed SBWTCK
- net SBWTCK: now also J1.6 (Pin_6); no longer J1.5 (Pin_5)
Changed lines of the file:
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@@
 		)
 	)
-	(label "SBTCK"
+	(label "SBWTCK"
 		(at 104.14 92.71 0)
 		(effects
@@
 		)
 	)
-	(label "SBWTDIO"
+	(label "SBWTCK"
 		(at 68.58 120.65 0)
 		(effects
@@
 		)
 	)
-	(label "SBTCK"
+	(label "SBWTDIO"
 		(at 68.58 118.11 0)
 		(effects
